Commit message: gazebo simulation

File: src/diffbot_description/urdf/diffbot.urdf.xacro (robot description, xacro)
@@ -1,6 +1,4 @@
 <?xml version="1.0"?>
 <robot xmlns:xacro="http://www.ros.org/wiki/xacro" name="diffbot">
-    <!-- INCLUDE INERTIAL MACROS -->
-    <xacro:include filename="inertial_macros.xacro"/>
     <!-- COLOR DEFINITIONS -->
     <material name="white">
@@ -11,9 +9,18 @@
     </material>
     <material name="blue">
-        <color rgba="0.2 0.2 1 1"/>
+        <color rgba="0 0 1 1"/>
     </material>
     <material name="black">
         <color rgba="0 0 0 1"/>
     </material>
+    <material name="brown">
+        <color rgba="0.7 0.55 0.3 1"/>
+    </material>
+    <!-- ________________________XACRO FILE DEPENDENCIES________________________ -->
+    <!-- INCLUDE INERTIAL MACROS -->
+    <xacro:include filename="$(find diffbot_description)/urdf/inertial_macros.xacro"/>
+    <!-- GAZEBO -->
+    <xacro:include filename="$(find diffbot_description)/urdf/diffbot_gazebo.xacro"/>
+    <!-- ________________________DIFFBOT URDF MODEL________________________ -->
     <!-- BASE LINK -->
     <link name="base_link"/>
@@ -30,5 +37,5 @@
                 <box size="0.3 0.22 0.08"/>
             </geometry>
-            <material name="white"/>
+            <material name="brown"/>
         </visual>
         <collision>

Commit message: kinematics and joystick control

File: src/diffbot_description/urdf/diffbot.urdf.xacro (robot description, xacro)
@@ -17,10 +17,15 @@
         <color rgba="0.7 0.55 0.3 1"/>
     </material>
-    <!-- ________________________XACRO FILE DEPENDENCIES________________________ -->
+    <!-- ________________________ ARGUMENT DEFINITIONS ________________________ -->
+    <!-- ROS2 VERSION -->
+    <xacro:arg name="is_ignition" default="true"/>
+    <!-- ________________________ XACRO FILE DEPENDENCIES ________________________ -->
     <!-- INCLUDE INERTIAL MACROS -->
     <xacro:include filename="$(find diffbot_description)/urdf/inertial_macros.xacro"/>
     <!-- GAZEBO -->
     <xacro:include filename="$(find diffbot_description)/urdf/diffbot_gazebo.xacro"/>
-    <!-- ________________________DIFFBOT URDF MODEL________________________ -->
+    <!-- ROS2 CONTROL -->
+    <xacro:include filename="$(find diffbot_description)/urdf/diffbot_ros2_control.xacro"/>
+    <!-- ________________________ DIFFBOT URDF MODEL ________________________ -->
     <!-- BASE LINK -->
     <link name="base_link"/>
@@ -45,5 +50,5 @@
             </geometry>
         </collision>
-        <xacro:inertial_box mass="0.5" x="0.3" y="0.3" z="0.15">
+        <xacro:inertial_box mass="0.5" x="0.3" y="0.22" z="0.08">
             <origin xyz="0 0 0" rpy="0 0 0"/>
         </xacro:inertial_box>
@@ -53,5 +58,5 @@
         <parent link="base_link"/>
         <child link="left_wheel"/>
-        <origin xyz="-0.075 0.1225 0" rpy="${-pi/2} 0 0"/>
+        <origin xyz="-0.075 0.1225 0" rpy="-${pi/2} 0 0" />
         <axis xyz="0 0 1"/>
     </joint>
@@ -77,5 +82,5 @@
         <child link="right_wheel"/>
         <origin xyz="-0.075 -0.1225 0" rpy="${pi/2} 0 0" />
-        <axis xyz="0 0 1"/>
+        <axis xyz="0 0 -1"/>
     </joint>
     <link name="right_wheel">

File: src/diffbot_description/urdf/diffbot_gazebo.xacro (robot description, xacro)
@@ -1,7 +1,10 @@
 <?xml version="1.0"?>
-<robot name="diffbot" xmlns:xacro="http//:www.ros.org/wiki/xacro">
-    <gazebo reference="left_wheel_joint">
-        <mu1>100000000000000.0</mu1>
-        <mu2>100000000000000.0</mu2>
+<robot name="diffbot" xmlns:xacro="http://www.ros.org/wiki/xacro">
+    <gazebo reference="left_wheel">
+        <visual>
+        <material name="blue"/>
+        </visual>
+        <mu1>1000000000000000.0</mu1>
+        <mu2>1000000000000000.0</mu2>
         <kp>1000000000000.0</kp>
         <kd>10.0</kd>
@@ -10,7 +13,10 @@
         <fdir1>1 0 0</fdir1>
     </gazebo>
-    <gazebo reference="right_wheel_joint">
-        <mu1>100000000000000.0</mu1>
-        <mu2>100000000000000.0</mu2>
+    <gazebo reference="right_wheel">
+        <visual>
+        <material name="blue"/>
+        </visual>
+        <mu1>1000000000000000.0</mu1>
+        <mu2>1000000000000000.0</mu2>
         <kp>1000000000000.0</kp>
         <kd>10.0</kd>
@@ -19,7 +25,7 @@
         <fdir1>1 0 0</fdir1>
     </gazebo>
-    <gazebo reference="caster_wheel_joint">
-        <mu1>0.1</mu1>
-        <mu2>0.1</mu2>
+    <gazebo reference="caster_wheel">
+        <mu1>0.001</mu1>
+        <mu2>0.001</mu2>
         <kp>1000000.0</kp>
         <kd>100.0</kd>
@@ -27,3 +33,15 @@
         <maxVel>0.1</maxVel>
     </gazebo>
+    <gazebo>
+        <xacro:if value="$(arg is_ignition)">
+            <plugin filename="ign_ros2_control-system" name="ign_ros2_control::IgnitionROS2ControlPlugin">
+                <parameters>$(find diffbot_controller)/config/diffbot_controllers.yaml</parameters>
+            </plugin>
+        </xacro:if>
+        <xacro:unless value="$(arg is_ignition)">
+            <plugin filename="gz_ros2_control-system" name="gz_ros2_control::GazeboSimROS2ControlPlugin">
+                <parameters>$(find diffbot_controller)/config/diffbot_controllers.yaml</parameters>
+            </plugin>
+        </xacro:unless>
+    </gazebo>
 </robot>

Commit message: firmware

File: src/diffbot_description/urdf/diffbot.urdf.xacro (robot description, xacro)
@@ -20,4 +20,6 @@
     <!-- ROS2 VERSION -->
     <xacro:arg name="is_ignition" default="true"/>
+    <!-- START SIMULATION OR REAL ROBOT -->
+    <xacro:arg name="is_sim" default="true"/>
     <!-- ________________________ XACRO FILE DEPENDENCIES ________________________ -->
     <!-- INCLUDE INERTIAL MACROS -->

File: src/diffbot_description/urdf/diffbot_ros2_control.xacro (robot description, xacro)
@@ -2,30 +2,41 @@
 <robot name="diffbot" xmlns:xacro="http//:www.ros.org/wiki/xacro">
     <ros2_control name="RobotSystem" type="system">
-        <xacro:if value="$(arg is_ignition)">
+        <!-- REAL ROBOT OR SIMULATION -->
+        <xacro:if value="$(arg is_sim)">
+            <!-- ROS2 VERSION -->
+            <xacro:if value="$(arg is_ignition)">
+                <hardware>
+                    <plugin>ign_ros2_control/IgnitionSystem</plugin>
+                </hardware>
+            </xacro:if>
+            <xacro:unless value="$(arg is_ignition)">
+                <hardware>
+                    <plugin>gz_ros2_control/GazeboSimSystem</plugin>
+                </hardware>
+            </xacro:unless>
+        </xacro:if>
+        <xacro:unless value="$(arg is_sim)">
             <hardware>
-                <plugin>ign_ros2_control/IgnitionSystem</plugin>
-            </hardware>
-        </xacro:if>
-        <xacro:unless value="$(arg is_ignition)">
-            <hardware>
-                <plugin>gz_ros2_control/GazeboSimSystem</plugin>
+                <plugin>diffbot_firmware/DiffbotInterface</plugin>
+                <param name="port">/dev/ttyACM0</param>
             </hardware>
         </xacro:unless>
-    <joint name="right_wheel_joint">
-        <command_interface name="velocity">
-            <param name="min">-1</param>
-            <param name="max">1</param>
-        </command_interface>
-        <state_interface name = "position"/>
-        <state_interface name = "velocity"/>
-    </joint>
-    <joint name="left_wheel_joint">
-        <command_interface name="velocity">
-            <param name="min">-1</param>
-            <param name="max">1</param>
-        </command_interface>
-        <state_interface name = "position"/>
-        <state_interface name = "velocity"/>
-    </joint>
+        <!-- ROS2 CONTROL CONFIGURATION -->
+        <joint name="right_wheel_joint">
+            <command_interface name="velocity">
+                <param name="min">-1</param>
+                <param name="max">1</param>
+            </command_interface>
+            <state_interface name = "position"/>
+            <state_interface name = "velocity"/>
+        </joint>
+        <joint name="left_wheel_joint">
+            <command_interface name="velocity">
+                <param name="min">-1</param>
+                <param name="max">1</param>
+            </command_interface>
+            <state_interface name = "position"/>
+            <state_interface name = "velocity"/>
+        </joint>
     </ros2_control>
 </robot>
