Commit message: robot working properly

File: diffbot_ws/src/diffbot_description/urdf/diffbot.urdf.xacro (robot description, xacro)
@@ -57,11 +57,11 @@
     </link>
     <!-- LEFT WHEEL -->
-    <joint name="left_wheel_joint" type="continuous">
+    <joint name="wheel_left_joint" type="continuous">
         <parent link="base_link"/>
-        <child link="left_wheel"/>
+        <child link="wheel_left"/>
         <origin xyz="-0.075 0.1225 0" rpy="-${pi/2} 0 0" />
         <axis xyz="0 0 1"/>
     </joint>
-    <link name="left_wheel">
+    <link name="wheel_left">
         <visual>
             <geometry>
@@ -80,11 +80,11 @@
     </link>
     <!-- RIGHT WHEEL -->
-    <joint name="right_wheel_joint" type="continuous">
+    <joint name="wheel_right_joint" type="continuous">
         <parent link="base_link"/>
-        <child link="right_wheel"/>
+        <child link="wheel_right"/>
         <origin xyz="-0.075 -0.1225 0" rpy="${pi/2} 0 0" />
         <axis xyz="0 0 -1"/>
     </joint>
-    <link name="right_wheel">
+    <link name="wheel_right">
         <visual>
             <geometry>
@@ -124,3 +124,32 @@
         </xacro:inertial_sphere>
     </link>
+    <!-- IMU -->
+    <link name="imu_link">
+        <inertial>
+            <origin xyz="0.0175 0.0175 0" rpy="0 0 0"/>
+            <mass value="0.000528415"/>
+            <inertia ixx="1.4617E-08" ixy="1.4E-10" ixz="-1.9963E-12"
+                    iyy="1.4617E-08" iyz="7.5237E-12"
+                    izz="2.3027E-08"/>
+        </inertial>
+        <visual>
+            <origin xyz="0.0175 0.0175 0" rpy="${pi/2} 0 ${pi}"/>
+            <geometry>
+                <mesh filename="package://diffbot_description/meshes/WT901C.stl"/>
+            </geometry>
+            <material name="black"/>
+        </visual>
+        <collision>
+            <origin xyz="0.0175 0.0175 0" rpy="0 0 0"/>
+            <geometry>
+                <mesh filename="package://diffbot_description/meshes/WT901C.stl"/>
+            </geometry>
+        </collision>
+    </link>
+    <joint name="imu_joint" type="fixed">
+        <origin xyz="${0.3/2 - 0.005 - 0.0175} ${0.22/2 - 0.025 - 0.0175} ${0.06+0.08/2}" rpy="0 0 0" />
+        <parent link="base_link"/>
+        <child link="imu_link"/>
+        <axis xyz="0 0 0"/>
+    </joint>
 </robot>

File: diffbot_ws/src/diffbot_description/urdf/diffbot_gazebo.xacro (robot description, xacro)
@@ -13,5 +13,5 @@
         <fdir1>1 0 0</fdir1>
     </gazebo>
-    <gazebo reference="right_wheel">
+    <gazebo reference="wheel_right">
         <visual>
         <material name="blue"/>
@@ -33,15 +33,64 @@
         <maxVel>0.1</maxVel>
     </gazebo>
-    <gazebo>
-        <xacro:if value="$(arg is_ignition)">
-            <plugin filename="ign_ros2_control-system" name="ign_ros2_control::IgnitionROS2ControlPlugin">
-                <parameters>$(find diffbot_controller)/config/diffbot_controllers.yaml</parameters>
-            </plugin>
-        </xacro:if>
-        <xacro:unless value="$(arg is_ignition)">
-            <plugin filename="gz_ros2_control-system" name="gz_ros2_control::GazeboSimROS2ControlPlugin">
-                <parameters>$(find diffbot_controller)/config/diffbot_controllers.yaml</parameters>
-            </plugin>
-        </xacro:unless>
+  <!-- ROS 2 Control -->
+  <gazebo>
+    <!-- ROS 2 Humble -->
+    <xacro:if value="$(arg is_ignition)">
+      <plugin filename="ign_ros2_control-system" name="ign_ros2_control::IgnitionROS2ControlPlugin">
+        <parameters>$(find diffbot_controller)/config/diffbot_controllers.yaml</parameters>
+      </plugin>
+      <plugin filename="ignition-gazebo-imu-system" name="ignition::gazebo::systems::Imu">
+      </plugin>
+    </xacro:if>
+  </gazebo>
+    <gazebo reference="imu_link">
+        <sensor name="imu" type="imu">
+            <always_on>true</always_on>
+            <update_rate>100</update_rate>
+            <gz_frame_id>imu_link</gz_frame_id>
+            <topic>imu</topic>
+            <imu>
+                <angular_velocity>
+                    <x>
+                        <noise type="gaussian">
+                            <mean>0.0</mean>
+                            <stddev>2e-4</stddev>
+                        </noise>
+                    </x>
+                    <y>
+                        <noise type="gaussian">
+                            <mean>0.0</mean>
+                            <stddev>2e-4</stddev>
+                        </noise>
+                    </y>
+                    <z>
+                        <noise type="gaussian">
+                            <mean>0.0</mean>
+                            <stddev>2e-4</stddev>
+                        </noise>
+                    </z>
+                </angular_velocity>
+                <linear_acceleration>
+                    <x>
+                        <noise type="gaussian">
+                            <mean>0.0</mean>
+                            <stddev>1.7e-2</stddev>
+                        </noise>
+                    </x>
+                    <y>
+                        <noise type="gaussian">
+                            <mean>0.0</mean>
+                            <stddev>1.7e-2</stddev>
+                        </noise>
+                    </y>
+                    <z>
+                        <noise type="gaussian">
+                            <mean>0.0</mean>
+                            <stddev>1.7e-2</stddev>
+                        </noise>
+                    </z>
+                </linear_acceleration>
+            </imu>
+        </sensor>
     </gazebo>
 </robot>

File: diffbot_ws/src/diffbot_description/urdf/diffbot_ros2_control.xacro (robot description, xacro)
@@ -1,8 +1,8 @@
 <?xml version="1.0"?>
-<robot name="diffbot" xmlns:xacro="http//:www.ros.org/wiki/xacro">
+<robot xmlns:xacro="http://www.ros.org/wiki/xacro" name="diffbot">
     <ros2_control name="RobotSystem" type="system">
-        <!-- REAL ROBOT OR SIMULATION -->
+        <!-- ros2_control Gazebo -->
         <xacro:if value="$(arg is_sim)">
-            <!-- ROS2 VERSION -->
+            <!-- ROS 2 Humble -->
             <xacro:if value="$(arg is_ignition)">
                 <hardware>
@@ -10,4 +10,5 @@
                 </hardware>
             </xacro:if>
+            <!-- ROS 2 Iron or above -->
             <xacro:unless value="$(arg is_ignition)">
                 <hardware>
@@ -16,26 +17,27 @@
             </xacro:unless>
         </xacro:if>
+        <!-- ros2_control Real Robot -->
         <xacro:unless value="$(arg is_sim)">
             <hardware>
                 <plugin>diffbot_firmware/DiffbotInterface</plugin>
-                <param name="port">/dev/ttyACM0</param>
+                <param name="port">/dev/ttyESP32</param>
             </hardware>
         </xacro:unless>
-        <!-- ROS2 CONTROL CONFIGURATION -->
-        <joint name="right_wheel_joint">
+        <!-- ros2_control Common Interfaces -->
+        <joint name="wheel_right_joint">
             <command_interface name="velocity">
-                <param name="min">-1</param>
-                <param name="max">1</param>
+              <param name="min">-1</param>
+              <param name="max">1</param>
             </command_interface>
-            <state_interface name = "position"/>
-            <state_interface name = "velocity"/>
+            <state_interface name="position" />
+            <state_interface name="velocity" />
         </joint>
-        <joint name="left_wheel_joint">
+        <joint name="wheel_left_joint">
             <command_interface name="velocity">
-                <param name="min">-1</param>
-                <param name="max">1</param>
+              <param name="min">-1</param>
+              <param name="max">1</param>
             </command_interface>
-            <state_interface name = "position"/>
-            <state_interface name = "velocity"/>
+            <state_interface name="position" />
+            <state_interface name="velocity" />
         </joint>
     </ros2_control>

Commit message: Odometry changes
- Kalman filter for sensor fusion
- Add imu to the simulation
- Fix python noisy controller

File: diffbot_ws/src/diffbot_description/urdf/diffbot.urdf.xacro (robot description, xacro)
@@ -124,3 +124,31 @@
         </xacro:inertial_sphere>
     </link>
+    <!-- IMU -->
+    <link name="imu_link">
+        <inertial>
+            <origin xyz="-0.0055 0.00016821 0.000514" rpy="0 0 0"/>
+                <mass value="0.000528415"/>
+                <inertia ixx="1.4617E-08" ixy="1.4E-10" ixz="-1.9963E-12"
+                        iyy="1.4617E-08" iyz="7.5237E-12"
+                        izz="2.3027E-08"/>
+        </inertial>
+        <visual>
+            <origin xyz="0 0 0" rpy="0 0 0"/>
+            <geometry>
+                <mesh filename="package://diffbot_description/meshes/imu_link.STL"/>
+            </geometry>
+        </visual>
+        <collision>
+            <origin xyz="0 0 0" rpy="0 0 0"/>
+            <geometry>
+                <mesh filename="package://diffbot_description/meshes/imu_link.STL"/>
+            </geometry>
+        </collision>
+    </link>
+    <joint name="imu_joint" type="fixed">
+        <origin xyz="0.075 0 0.07" rpy="0 0 0" />
+        <parent link="base_link"/>
+        <child link="imu_link"/>
+        <axis xyz="0 0 0"/>
+    </joint>
 </robot>

File: diffbot_ws/src/diffbot_description/urdf/diffbot_gazebo.xacro (robot description, xacro)
@@ -38,4 +38,6 @@
                 <parameters>$(find diffbot_controller)/config/diffbot_controllers.yaml</parameters>
             </plugin>
+            <plugin filename="ignition-gazebo-imu-system" name="ignition::gazebo::systems::Imu">
+            </plugin>
         </xacro:if>
         <xacro:unless value="$(arg is_ignition)">
@@ -43,5 +45,57 @@
                 <parameters>$(find diffbot_controller)/config/diffbot_controllers.yaml</parameters>
             </plugin>
+            <plugin filename="gz-sim-imu-system" name="g::sim::system::Imu">
+            </plugin>
         </xacro:unless>
     </gazebo>
+    <gazebo reference="imu_link">
+        <sensor name="imu" type="imu">
+            <always_on>true</always_on>
+            <update_rate>100</update_rate>
+            <gz_frame_id>imu_link</gz_frame_id>
+            <topic>imu</topic>
+            <imu>
+                <angular_velocity>
+                    <x>
+                        <noise type="gaussian">
+                            <mean>0.0</mean>
+                            <stddev>2e-4</stddev>
+                        </noise>
+                    </x>
+                    <y>
+                        <noise type="gaussian">
+                            <mean>0.0</mean>
+                            <stddev>2e-4</stddev>
+                        </noise>
+                    </y>
+                    <z>
+                        <noise type="gaussian">
+                            <mean>0.0</mean>
+                            <stddev>2e-4</stddev>
+                        </noise>
+                    </z>
+                </angular_velocity>
+                <linear_acceleration>
+                    <x>
+                        <noise type="gaussian">
+                            <mean>0.0</mean>
+                            <stddev>1.7e-2</stddev>
+                        </noise>
+                    </x>
+                    <y>
+                        <noise type="gaussian">
+                            <mean>0.0</mean>
+                            <stddev>1.7e-2</stddev>
+                        </noise>
+                    </y>
+                    <z>
+                        <noise type="gaussian">
+                            <mean>0.0</mean>
+                            <stddev>1.7e-2</stddev>
+                        </noise>
+                    </z>
+                </linear_acceleration>
+            </imu>
+        </sensor>
+    </gazebo>
 </robot>

Commit message: robot localization (simulation)

File: diffbot_ws/src/diffbot_description/urdf/diffbot.urdf.xacro (robot description, xacro)
@@ -147,5 +147,5 @@
     </link>
     <joint name="imu_joint" type="fixed">
-        <origin xyz="0.075 0 0.07" rpy="0 0 0" />
+        <origin xyz="0.125 0.065 0.105" rpy="0 0 0" />
         <parent link="base_link"/>
         <child link="imu_link"/>

Commit message: imu configuration
- modify the urdf.xacro to include the imu
- adapt the robot_localization launcher to use the imu topic as a parameter

File: diffbot_ws/src/diffbot_description/urdf/diffbot.urdf.xacro (robot description, xacro)
@@ -127,25 +127,26 @@
     <link name="imu_link">
         <inertial>
-            <origin xyz="-0.0055 0.00016821 0.000514" rpy="0 0 0"/>
-                <mass value="0.000528415"/>
-                <inertia ixx="1.4617E-08" ixy="1.4E-10" ixz="-1.9963E-12"
-                        iyy="1.4617E-08" iyz="7.5237E-12"
-                        izz="2.3027E-08"/>
+            <origin xyz="0.0175 0.0175 0" rpy="0 0 0"/>
+            <mass value="0.000528415"/>
+            <inertia ixx="1.4617E-08" ixy="1.4E-10" ixz="-1.9963E-12"
+                    iyy="1.4617E-08" iyz="7.5237E-12"
+                    izz="2.3027E-08"/>
         </inertial>
         <visual>
-            <origin xyz="0 0 0" rpy="0 0 0"/>
+            <origin xyz="0.0175 0.0175 0" rpy="${pi/2} 0 ${pi}"/>
             <geometry>
-                <mesh filename="package://diffbot_description/meshes/imu_link.STL"/>
+                <mesh filename="package://diffbot_description/meshes/WT901C.stl"/>
             </geometry>
+            <material name="black"/>
         </visual>
         <collision>
-            <origin xyz="0 0 0" rpy="0 0 0"/>
+            <origin xyz="0.0175 0.0175 0" rpy="0 0 0"/>
             <geometry>
-                <mesh filename="package://diffbot_description/meshes/imu_link.STL"/>
+                <mesh filename="package://diffbot_description/meshes/WT901C.stl"/>
             </geometry>
         </collision>
     </link>
     <joint name="imu_joint" type="fixed">
-        <origin xyz="0.125 0.065 0.105" rpy="0 0 0" />
+        <origin xyz="${0.3/2 - 0.005 - 0.0175} ${0.22/2 - 0.025 - 0.0175} ${0.06+0.08/2}" rpy="0 0 0" />
         <parent link="base_link"/>
         <child link="imu_link"/>

Commit message: fix imu collision problem

File: diffbot_ws/src/diffbot_description/urdf/diffbot.urdf.xacro (robot description, xacro)
@@ -126,11 +126,7 @@
     <!-- IMU -->
     <link name="imu_link">
-        <inertial>
-            <origin xyz="0.0175 0.0175 0" rpy="0 0 0"/>
-            <mass value="0.000528415"/>
-            <inertia ixx="1.4617E-08" ixy="1.4E-10" ixz="-1.9963E-12"
-                    iyy="1.4617E-08" iyz="7.5237E-12"
-                    izz="2.3027E-08"/>
-        </inertial>
+        <xacro:inertial_box mass="0.006" x="0.035" y="0.035" z="0.015">
+            <origin xyz="0 0 0.003" rpy="0 0 0"/>
+        </xacro:inertial_box>
         <visual>
             <origin xyz="0.0175 0.0175 0" rpy="${pi/2} 0 ${pi}"/>
@@ -141,5 +137,5 @@
         </visual>
         <collision>
-            <origin xyz="0.0175 0.0175 0" rpy="0 0 0"/>
+            <origin xyz="0.0175 0.0175 0" rpy="${pi/2} 0 ${pi}"/>
             <geometry>
                 <mesh filename="package://diffbot_description/meshes/WT901C.stl"/>

Commit message: starting with nav2: use a twist mux and add a lifecycle manager and map server

File: diffbot_ws/src/diffbot_description/urdf/diffbot.urdf.xacro (robot description, xacro)
@@ -149,3 +149,30 @@
         <axis xyz="0 0 0"/>
     </joint>
+    <!-- LIDAR -->
+    <link name="laser_link">
+        <inertial>
+            <origin xyz="-0.011945780406062 -0.000381929217680526 -0.0170649378129477" rpy="0 0 0" />
+            <mass value="0.073084435549317" />
+            <inertia ixx="1.96074931730795E-05" ixy="-3.62091076640009E-07" ixz="4.28230084046735E-07" iyy="2.40983835136327E-05" iyz="1.50180909250652E-08" izz="4.14184164228595E-05" />
+        </inertial>
+        <visual>
+            <origin xyz="0 0 0" rpy="0 0 0"/>
+            <geometry>
+                <mesh filename="package://diffbot_description/meshes/laser_link.STL"/>
+            </geometry>
+            <material name="black"/>
+        </visual>
+        <collision>
+            <origin xyz="0 0 0" rpy="0 0 0"/>
+            <geometry>
+                <mesh filename="package://diffbot_description/meshes/laser_link.STL"/>
+            </geometry>
+        </collision>
+    </link>
+    <joint name="laser_joint" type="fixed">
+        <origin xyz="0 0 ${0.08 + 0.06}" rpy="0 0 3.14" />
+        <parent link="base_link"/>
+        <child link="laser_link"/>
+        <axis xyz="0 0 0"/>
+    </joint>
 </robot>

File: diffbot_ws/src/diffbot_description/urdf/diffbot_gazebo.xacro (robot description, xacro)
@@ -41,4 +41,7 @@
       </plugin>
       <plugin filename="ignition-gazebo-imu-system" name="ignition::gazebo::systems::Imu">
+      </plugin>
+      <plugin filename="ignition-gazebo-sensors-system" name="ignition::gazebo::systems::Sensors">
+        <render_engine>ogre2</render_engine>
       </plugin>
     </xacro:if>
@@ -94,3 +97,32 @@
         </sensor>
     </gazebo>
+    <gazebo reference="laser_link">
+        <sensor name="lidar" type="gpu_ray">
+            <always_on>true</always_on>
+            <visualize>true</visualize>
+            <topic>scan</topic>
+            <update_rate>5</update_rate>
+            <gz_frame_id>laser_link</gz_frame_id>
+            <ray>
+                <scan>
+                    <horizontal>
+                        <samples>360</samples>
+                        <resolution>1.0</resolution>
+                        <min_angle>0.0</min_angle>
+                        <max_angle>6.28</max_angle>
+                    </horizontal>
+                </scan>
+                <range>
+                    <min>0.12</min>
+                    <max>2.0</max>
+                    <resolution>0.02</resolution>
+                </range>
+                <noise>
+                    <type>gaussian</type>
+                    <mean>0.0</mean>
+                    <stddev>0.01</stddev>
+                </noise>
+            </ray>
+        </sensor>
+    </gazebo>
 </robot>

Commit message: nav2

File: diffbot_ws/src/diffbot_description/urdf/diffbot.urdf.xacro (robot description, xacro)
@@ -132,5 +132,5 @@
             <origin xyz="0.0175 0.0175 0" rpy="${pi/2} 0 ${pi}"/>
             <geometry>
-                <mesh filename="package://diffbot_description/meshes/WT901C.stl"/>
+                <mesh filename="package://diffbot_description/meshes/WT901C.STL"/>
             </geometry>
             <material name="black"/>
@@ -139,5 +139,5 @@
             <origin xyz="0.0175 0.0175 0" rpy="${pi/2} 0 ${pi}"/>
             <geometry>
-                <mesh filename="package://diffbot_description/meshes/WT901C.stl"/>
+                <mesh filename="package://diffbot_description/meshes/WT901C.STL"/>
             </geometry>
         </collision>
